File: KiCAD/SmartWatch.kicad_pcb (KiCad board)
At the start: 4 copper layers, 35.6 x 35.6 mm, 89 parts

Commit message: Finished PCB
Parts:
- BT1: value (none) -> LiPoly 1S1P
- P1: value (none) -> CONN_6
- Q1: value (none) -> MMBT2222A
- SW1, SW2, SW3, SW4: value (none) -> SW_PUSH
- TP1, TP10, TP11, TP2, TP3, TP4, TP5, TP6, TP7, TP8, TP9: value (none) -> TP
- U1: value (none) -> BQ25010
- U2: value (none) -> MIC2290
- U3: value (none) -> FT201X
- U4: value (none) -> EROLED015-1
- U5: value (none) -> FXOS8700CQ
- U6: value (none) -> PIC32MX370F512H
- X1: value (none) -> 25MHz
- X2: value (none) -> 32.768KHz
- moved C15 24.7 mm to (233.5, 154.2)
- moved C16 22.3 mm to (231.5, 150.6), turned to 0 degrees
- moved C25 17.3 mm to (213.8, 149.6), turned to 270 degrees
- moved C17 16.8 mm to (228.5, 150.0), turned to 180 degrees
- moved C26 15.9 mm to (215.1, 149.6), turned to 270 degrees
- moved C24 11.7 mm to (216.5, 149.6), turned to 270 degrees
- moved C18 10.4 mm to (226.2, 149.4), turned to 270 degrees
- moved R12 7.65 mm to (217.9, 149.7), turned to 90 degrees
- moved U4 0.09 mm to (221.5, 152.8)
Routing:
- net /LCD/Sensors/D6: track 21.2 -> 7.19 mm
- net /LCD/Sensors/D5: track 19.2 -> 6.34 mm
- net /LCD/Sensors/D4: track 18.4 -> 6.87 mm
- net /LCD/Sensors/D7: track 23.0 -> 11.9 mm
- net GND: track 289.2 -> 279.7 mm, vias 69 -> 74
- net /LCD/Sensors/D3: track 15.4 -> 7.30 mm
- net /SW1: track 54.6 -> 62.0 mm
- net /USB/Power/Boost-En: track 42.6 -> 49.0 mm
- net /LCD/Sensors/R/W: track 16.5 -> 11.0 mm
- net /LCD/Sensors/D/C: track 27.2 -> 32.5 mm
- net +3.3V: track 94.7 -> 90.6 mm, vias 27 -> 28
- net /LCD/Sensors/D2: track 11.8 -> 7.70 mm
- net /USB/Power/nPG: track 22.6 -> 25.7 mm
- net /LCD/Sensors/E: track 16.6 -> 14.2 mm
- net /LCD/Sensors/D1: track 10.1 -> 8.16 mm
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- added copper zone on B.Cu, net +3.3V
- added copper zone on B.Cu, net GND
- added copper zone on F.Cu, net N-0000066
- removed copper zone on F.Cu, net N-0000063
Other:
- board text added: "Daniel A. 6/27/16"
- board text added: "GND"
- board text added: "VBAT"
- board text added: "bit.ly/2925hox"
- board text removed: "Daniel A. 6/24/16"

Commit message: Updated PCB
Routing:
- net GND: track 279.7 -> 290.5 mm, vias 74 -> 72
