File: KiCAD/SmartWatch.kicad_pcb (KiCad board)
At the start: 4 copper layers, 35.6 x 35.6 mm, 89 parts, among them P1 CONN_6, Q1 MMBT2222A, SW1 SW_PUSH, SW2 SW_PUSH, SW3 SW_PUSH, SW4 SW_PUSH, U1 BQ25010, U2 MIC2290, U3 FT201X, U4 EROLED015-1, U5 FXOS8700CQ, U6 PIC32MX370F512H, X1 25MHz, X2 32.768KHz

Commit message: Finished PCB Rev 2.0
Parts:
- C17: footprint c_0805 -> c_1206
- moved C3 11.7 mm to (205.0, 142.9)
- moved R2 10.0 mm to (214.0, 146.4), turned to 90 degrees
- moved R3 9.92 mm to (215.4, 146.4), turned to 270 degrees
- moved R1 9.85 mm to (212.6, 146.4), turned to 90 degrees
- moved I1 6.99 mm to (206.0, 139.6), turned to 0 degrees
- moved C4 6.93 mm to (206.0, 146.7), turned to 90 degrees
- moved R4 5.54 mm to (207.4, 146.9), turned to 270 degrees
- moved R5 4.43 mm to (208.8, 147.3), turned to 270 degrees
- moved C5 3.82 mm to (210.2, 147.6), turned to 90 degrees
- moved U1 2.91 mm to (209.6, 142.7), turned to 0 degrees
- moved C1 1.13 mm to (209.2, 150.0)
- moved C16 1.05 mm to (232.5, 150.4), turned to 270 degrees
- moved C17 1.00 mm to (229.5, 150.4)
- moved C6 0.56 mm to (205.9, 149.7)
Connections:
- X1 pad 3: (no net) -> GND
- X1 pad 4: (no net) -> GND
Routing:
- net +3.3V: track 90.6 -> 103.3 mm, vias 28 -> 31
- net /USB/Power/USB +5V: track 48.2 -> 40.7 mm
- net N-0000072: track 4.06 -> 9.49 mm
- net /USB/Power/nPG: track 25.7 -> 20.9 mm
- net GND: track 290.5 -> 295.2 mm, vias 72 -> 86
- net /USB/Power/STAT1: track 24.5 -> 20.8 mm, vias 2 -> 4
- net N-0000065: track 2.63 -> 0.00 mm
- net N-0000073: track 3.73 -> 5.71 mm
- net /USB/Power/FTDI_RST: track 57.7 -> 59.1 mm
- net /SW1: track 62.0 -> 63.3 mm
- net /SW4: track 22.8 -> 23.6 mm
- net VBAT: track 85.6 -> 86.3 mm
- net /USB/Power/Boost-En: track 49.0 -> 49.7 mm
- net +13V: track 36.7 -> 36.0 mm
- net /USB/Power/STAT2: track 25.9 -> 25.2 mm
- removed copper zone on F.Cu, net N-0000066
Other:
- board text added: "Daniel A. 7/19/16"
- board text added: "REV 2.0"
